Commit message: Update URDF dimensions to match measured robot hardware
- base body: 0.179×0.165×0.022 → 0.23×0.180×0.055 m
- wheel_radius: 0.032375 → 0.033 m
- wheel_width: 0.058 → 0.015 m
- Add wheel_track (0.160 m) and wheel_x_offset (0.0785 m) properties
- Fix wheel joint z: was -wheel_radius (axle underground), now 0 (correct)
- Wheel y now uses wheel_track/2 instead of base_width/2 + wheel_width/2
- laser_frame position unchanged

Co-Authored-By: Claude Sonnet 4.6 <noreply@anthropic.com>

File: urdf/robot_core.xacro (robot description, xacro)
@@ -2,9 +2,12 @@
 <robot xmlns:xacro="http://www.ros.org/wiki/xacro">
     <!-- Define some properties (easy to change later) -->
-    <xacro:property name="base_width" value="0.165"/>
-    <xacro:property name="base_length" value="0.179"/>
-    <xacro:property name="base_height" value="0.022"/>
-    <xacro:property name="wheel_radius" value="0.032375"/>
-    <xacro:property name="wheel_width" value="0.058"/>
+    <xacro:property name="base_width" value="0.180"/>
+    <xacro:property name="base_length" value="0.23"/>
+    <xacro:property name="base_height" value="0.055"/>
+    <xacro:property name="wheel_radius" value="0.033"/>
+    <xacro:property name="wheel_width" value="0.015"/>
+    <!-- wheel_track: center-to-center lateral distance; wheel_x_offset: forward from body center -->
+    <xacro:property name="wheel_track" value="0.160"/>
+    <xacro:property name="wheel_x_offset" value="0.0785"/>
     <!-- Materials for visualization -->
     <material name="white">
@@ -91,5 +94,5 @@
         <parent link="base_link"/>
         <child link="left_wheel"/>
-        <origin xyz="0 ${base_width/2 + wheel_width/2} -${wheel_radius}" rpy="0 0 0"/>
+        <origin xyz="${wheel_x_offset} ${wheel_track/2} 0" rpy="0 0 0"/>
         <axis xyz="0 1 0"/>
     </joint>
@@ -97,5 +100,5 @@
         <parent link="base_link"/>
         <child link="right_wheel"/>
-        <origin xyz="0 -${base_width/2 + wheel_width/2} -${wheel_radius}" rpy="0 0 0"/>
+        <origin xyz="${wheel_x_offset} -${wheel_track/2} 0" rpy="0 0 0"/>
         <axis xyz="0 1 0"/>
     </joint>
