Commit message: Fix lidar orientation (rotated 180 degrees)
The RPLIDAR was showing scan data 180 degrees off from the robot's
actual orientation. Added pi rotation to laser_frame joint.

https://claude.ai/code/session_01DWDVgLkdm56Xs1ttrUjox1

File: urdf/lidar.xacro (robot description, xacro)
@@ -31,5 +31,5 @@
         <parent link="base_link"/>
         <child link="laser_frame"/>
-        <origin xyz="${lidar_x_offset} ${lidar_y_offset} ${lidar_z_offset}" rpy="0 0 0"/>
+        <origin xyz="${lidar_x_offset} ${lidar_y_offset} ${lidar_z_offset}" rpy="0 0 ${pi}"/>
     </joint>
     <gazebo reference="laser_frame">
